File: clock-module-555-v2.kicad_pcb (KiCad board)
At the start: 2 copper layers, 65 x 50.1 mm, 37 parts, among them J1 Conn_01x03_Pin, J2 Conn_01x03_Socket, SW1 MODE, SW2 PULSE, U1 NE555P, U2 74HC112, U3 NE555P, U4 74HC00, U5 NE555P

Commit message: revisions after first build
Parts:
- C12: value 100nF -> 1uF
- RV1: value 100K -> 1M
- moved C13 2.02 mm to (85.5, 35.0), turned to 0 degrees
Connections:
- C13 pad 1: GND -> VCC
- C13 pad 2: VCC -> GND

Commit message: marked as rev 2
Other:
- board text added: "Rev 2"
Changed lines of the file:
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@@
+		)
+	)
+	(gr_text "Rev 2"
+		(at 35.4 27.4 0)
+		(layer "B.SilkS")
+		(effects
+			(font
+				(size 1 1)
+				(thickness 0.15)
+			)
+			(justify left bottom mirror)
 		)
 	)
