File: clock-module-555-v2.kicad_sch (KiCad schematic)
At the start: 37 parts, among them J1 Conn_01x03_Pin, J2 Conn_01x03_Socket, SW1 MODE, SW2 PULSE, U1 NE555P, U2 74HC112, U3 NE555P, U4 74HC00, U5 NE555P

Commit message: revisions after first build
Parts:
- C12: value 100nF -> 1uF
- C13: symbol Device:C_Polarized -> Device:C_Polarized_US
- RV1: value 100K -> 1M
Connections:
- net GND: now also C13.2; no longer C13.1
- net VCC: now also C13.1; no longer C13.2
Changed lines of the file:
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@@
 	)
 	(symbol
-		(lib_id "Device:C_Polarized")
-		(at 240.03 36.83 180)
+		(lib_id "Device:C_Polarized_US")
+		(at 240.03 36.83 0)
 		(unit 1)
 		(exclude_from_sim no)
@@
 		(fields_autoplaced yes)
 		(property "Reference" "C13"
-			(at 243.84 36.449 0)
-			(effects
-				(font
-					(size 1.27 1.27)
-				)
-				(justify right)
+			(at 243.84 34.9249 0)
+			(effects
+				(font
+					(size 1.27 1.27)
+				)
+				(justify left)
 			)
 		)
 		(property "Value" "1uF"
-			(at 243.84 38.989 0)
-			(effects
-				(font
-					(size 1.27 1.27)
-				)
-				(justify right)
+			(at 243.84 37.4649 0)
+			(effects
+				(font
+					(size 1.27 1.27)
+				)
+				(justify left)
 			)
 		)
 		(property "Footprint" "Capacitor_THT:CP_Radial_D5.0mm_P2.00mm"
-			(at 239.0648 33.02 0)
+			(at 240.03 36.83 0)
 			(effects
 				(font
@@
 			)
 		)
-		(property "Description" ""
+		(property "Description" "Polarized capacitor, US symbol"
 			(at 240.03 36.83 0)
 			(effects
@@
 		(fields_autoplaced yes)
 		(property "Reference" "C12"
-			(at 186.436 128.2763 0)
-			(effects
-				(font
-					(size 1.27 1.27)
-				)
-				(justify left)
-			)
-		)
-		(property "Value" "100nF"
-			(at 186.436 130.8163 0)
+			(at 185.42 128.2762 0)
+			(effects
+				(font
+					(size 1.27 1.27)
+				)
+				(justify left)
+			)
+		)
+		(property "Value" "1uF"
+			(at 185.42 130.8162 0)
 			(effects
 				(font
@@
 		(fields_autoplaced yes)
 		(property "Reference" "RV1"
-			(at 192.024 113.03 0)
+			(at 191.77 113.0299 0)
 			(effects
 				(font
@@
 			)
 		)
-		(property "Value" "100K"
-			(at 192.024 115.57 0)
-			(effects
-				(font
+		(property "Value" "1M"
+			(at 191.77 115.5699 0)
+			(effects
+				(font

Commit message: marked as rev 2
Other:
- moved on the sheet: C13, D2, H1, H2, H3, H4, J1, J2, R8, U2B, U4B, U4C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
